File: S2/C19/S2C19ST7D/S2C19ST7D.kicad_sch (KiCad schematic)
At the start: 3 parts

Commit message: upload S2 Chapter 19
Parts:
- L1: value 500m -> 10
- R1: value 10k -> 10
- V1: value 25 -> ${SIM.PARAMS}
