File: S2/C19/S2C19ST7E/S2C19ST7E.kicad_sch (KiCad schematic)
At the start: 3 parts

Commit message: upload S2 Chapter 19
Parts:
- L1: value 500m -> 1
- R1: value 10k -> 1k
- V1: value 25 -> ${SIM.PARAMS}
